Commit message: testes no gazebo e resolução de cmake e package

File: src/spot_robot/spot_description/urdf/spot_with_arm.urdf (robot description, URDF)
Before this commit: robot spot, 20 links, 19 joints
Links:
- link base: mass None -> 16.70765207

Commit message: mudanças spot_gazebo e tentativa de passar o robo setado no moveit no rviz

File: src/spot_robot/spot_description/urdf/spot_with_arm.urdf (robot description, URDF)
Before this commit: robot spot, 20 links, 19 joints
Links:
- removed link arm0.link_el0
- removed link arm0.link_el1
- removed link arm0.link_fngr
- removed link arm0.link_sh0
- removed link arm0.link_sh1
- removed link arm0.link_wr0
- removed link arm0.link_wr1
- removed link fl.hip
- removed link fl.lleg
- removed link fl.uleg
- removed link fr.hip
- removed link fr.lleg
- removed link fr.uleg
- removed link hl.hip
- removed link hl.lleg
- removed link hl.uleg
- removed link hr.hip
- removed link hr.lleg
- removed link hr.uleg
- added link arm0_link_el0, mass 0.94831958; collision mesh filename=package://spot_description/meshes/arm0_link_el0.stl; visual mesh filename=package://spot_description/meshes/arm0_link_el0.stl
- added link arm0_link_el1, mass 1.01754820; collision mesh filename=package://spot_description/meshes/arm0_link_el1.stl; visual mesh filename=package://spot_description/meshes/arm0_link_el1.stl
- added link arm0_link_fngr, mass 0.22383315; collision mesh filename=package://spot_description/meshes/arm0_link_fngr.stl; visual mesh filename=package://spot_description/meshes/arm0_link_fngr.stl
- added link arm0_link_sh0, mass 1.904699; collision mesh filename=package://spot_description/meshes/arm0_link_sh0.stl; visual mesh filename=package://spot_description/meshes/arm0_link_sh0.stl
- added link arm0_link_sh1, mass 1.85701942; collision mesh filename=package://spot_description/meshes/arm0_link_hr0.stl; collision mesh filename=package://spot_description/meshes/arm0_link_sh1.stl
- added link arm0_link_wr0, mass 0.58263740; collision mesh filename=package://spot_description/meshes/arm0_link_wr0.stl; visual mesh filename=package://spot_description/meshes/arm0_link_wr0.stl
- added link arm0_link_wr1, mass 0.93335298; collision mesh filename=package://spot_description/meshes/arm0_link_wr1.stl; visual mesh filename=package://spot_description/meshes/arm0_link_wr1.stl
- added link fl_hip, mass 1.13688339; collision mesh filename=package://spot_description/meshes/fl_hip_0_geom_visual_mesh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; visual mesh filename=package://spot_description/meshes/fl_hip_0_geom_visual_mesh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
- added link fl_lleg, mass 0.330; collision cylinder length=0.03 radius=0.033; collision cylinder length=0.35 radius=0.015
- added link fl_uleg, mass 2.25620359; collision cylinder length=0.35 radius=0.045; visual mesh filename=package://spot_description/meshes/l_uleg_0_geom_visual_mesh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
- added link fr_hip, mass 1.13688339; collision mesh filename=package://spot_description/meshes/fr_hip_0_geom_visual_mesh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; visual mesh filename=package://spot_description/meshes/fr_hip_0_geom_visual_mesh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
- added link fr_lleg, mass 0.330; collision cylinder length=0.03 radius=0.033; collision cylinder length=0.35 radius=0.015
- added link fr_uleg, mass 2.25620359; collision cylinder length=0.35 radius=0.045; visual mesh filename=package://spot_description/meshes/r_uleg_0_geom_visual_mesh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
- added link hl_hip, mass 1.13688339; collision mesh filename=package://spot_description/meshes/hl_hip_0_geom_visual_mesh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; visual mesh filename=package://spot_description/meshes/hl_hip_0_geom_visual_mesh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
- added link hl_lleg, mass 0.330; collision cylinder length=0.03 radius=0.033; collision cylinder length=0.35 radius=0.015
- added link hl_uleg, mass 2.25620359; collision cylinder length=0.35 radius=0.045; visual mesh filename=package://spot_description/meshes/l_uleg_0_geom_visual_mesh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
- added link hr_hip, mass 1.13688339; collision mesh filename=package://spot_description/meshes/hr_hip_0_geom_visual_mesh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; visual mesh filename=package://spot_description/meshes/hr_hip_0_geom_visual_mesh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
- added link hr_lleg, mass 0.330; collision cylinder length=0.03 radius=0.033; collision cylinder length=0.35 radius=0.015
- added link hr_uleg, mass 2.25620359; collision cylinder length=0.35 radius=0.045; visual mesh filename=package://spot_description/meshes/r_uleg_0_geom_visual_mesh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
Joints:
- removed joint arm0.el0
- removed joint arm0.el1
- removed joint arm0.f1x
- removed joint arm0.sh0
- removed joint arm0.sh1
- removed joint arm0.wr0
- removed joint arm0.wr1
- removed joint fl.hx
- removed joint fl.hy
- removed joint fl.kn
- removed joint fr.hx
- removed joint fr.hy
- removed joint fr.kn
- removed joint hl.hx
- removed joint hl.hy
- removed joint hl.kn
- removed joint hr.hx
- removed joint hr.hy
- removed joint hr.kn
- added joint arm0_el0: type revolute, parent arm0_link_sh1, child arm0_link_el0, origin xyz=0.3385 0 0, axis 0 1 0, limit lower=0 upper=3.14159 effort=90.9 velocity=999
- added joint arm0_el1: type revolute, parent arm0_link_el0, child arm0_link_el1, origin xyz=0.40330 0.0 0.0750, axis 1 0 0, limit lower=-2.792530 upper=2.792530 effort=30.3 velocity=999
- added joint arm0_f1x: type revolute, parent arm0_link_wr1, child arm0_link_fngr, origin xyz=0.11745 0 0.014820, axis 0 1 0, limit lower=-1.5708 upper=0.0 effort=15.32 velocity=999
- added joint arm0_sh0: type revolute, parent base, child arm0_link_sh0, origin xyz=0.292 0.0 0.188, axis 0 0 1, limit lower=-2.61799 upper=3.14159 effort=90.9 velocity=999
- added joint arm0_sh1: type revolute, parent arm0_link_sh0, child arm0_link_sh1, origin xyz=0.0 0.0 0.0, axis 0 1 0, limit lower=-3.14159 upper=0.523599 effort=181.8 velocity=999
- added joint arm0_wr0: type revolute, parent arm0_link_el1, child arm0_link_wr0, axis 0 1 0, limit lower=-1.8326 upper=1.8326 effort=30.3 velocity=999
- added joint arm0_wr1: type revolute, parent arm0_link_wr0, child arm0_link_wr1, axis 1 0 0, limit lower=-2.87989 upper=2.87979 effort=30.3 velocity=999
- added joint fl_hx: type revolute, parent base, child fl_hip, origin xyz=0.29785 0.05500 0.00000, axis 1 0 0, limit lower=-0.785398 upper=0.785398 effort=45 velocity=100
- added joint fl_hy: type revolute, parent fl_hip, child fl_uleg, origin xyz=0.0 0.110945 0.0, axis 0 1 0, limit lower=-0.898845 upper=2.295108 effort=45 velocity=100
- added joint fl_kn: type revolute, parent fl_uleg, child fl_lleg, origin xyz=0.025 0.000 -0.3205, axis 0 1 0, limit lower=-2.7929 upper=-0.2471 effort=115 velocity=100
- added joint fr_hx: type revolute, parent base, child fr_hip, origin xyz=0.29785 -0.05500 0.00000, axis 1 0 0, limit lower=-0.785398 upper=0.785398 effort=45 velocity=100
- added joint fr_hy: type revolute, parent fr_hip, child fr_uleg, origin xyz=0.0 -0.110945 0.0, axis 0 1 0, limit lower=-0.898845 upper=2.295108 effort=45 velocity=100
- added joint fr_kn: type revolute, parent fr_uleg, child fr_lleg, origin xyz=0.025 0.000 -0.3205, axis 0 1 0, limit lower=-2.7929 upper=-0.2471 effort=115 velocity=100
- added joint hl_hx: type revolute, parent base, child hl_hip, origin xyz=-0.29785 0.05500 0.00000, axis 1 0 0, limit lower=-0.785398 upper=0.785398 effort=45 velocity=100
- added joint hl_hy: type revolute, parent hl_hip, child hl_uleg, origin xyz=0.0 0.110945 0.0, axis 0 1 0, limit lower=-0.898845 upper=2.295108 effort=45 velocity=100
- added joint hl_kn: type revolute, parent hl_uleg, child hl_lleg, origin xyz=0.025 0.000 -0.3205, axis 0 1 0, limit lower=-2.7929 upper=-0.2471 effort=115 velocity=100
- added joint hr_hx: type revolute, parent base, child hr_hip, origin xyz=-0.29785 -0.05500 0.00000, axis 1 0 0, limit lower=-0.785398 upper=0.785398 effort=45 velocity=100
- added joint hr_hy: type revolute, parent hr_hip, child hr_uleg, origin xyz=0.0 -0.110945 0.0, axis 0 1 0, limit lower=-0.898845 upper=2.295108 effort=45 velocity=100
- added joint hr_kn: type revolute, parent hr_uleg, child hr_lleg, origin xyz=0.025 0.000 -0.3205, axis 0 1 0, limit lower=-2.7929 upper=-0.2471 effort=115 velocity=100

File: src/spot_robot/spot_moveit_config/config/spot.urdf.xacro (robot description, xacro)
@@ -2,8 +2,6 @@
 <robot xmlns:xacro="http://www.ros.org/wiki/xacro" name="spot">
     <xacro:arg name="initial_positions_file" default="initial_positions.yaml" />
-    <!-- Import spot urdf file -->
+    <!-- Importar a URDF do Spot -->
     <xacro:include filename="$(find spot_description)/urdf/spot_with_arm.urdf" />
-    <!-- Import control_xacro -->
-    <xacro:include filename="spot.ros2_control.xacro" />
-    <xacro:spot_ros2_control name="FakeSystem" initial_positions_file="$(arg initial_positions_file)"/>
+    <!-- Removemos o controle do ROS 2 -->
 </robot>
